File: fram-prototype.kicad_pcb (KiCad board)
At the start: 2 copper layers, 91.4 x 66 mm, 12 parts, among them J1 Barrel_Jack, SW1 Rotary_Encoder_Switch, U2 MAX6951

Commit message: first basic prototype
Parts:
- added C1: 10u, Capacitor_SMD:C_1206_3216Metric_Pad1.33x1.80mm_HandSolder, F.Cu at (67.3, 69.8)
- added C2: 22u, Capacitor_SMD:C_1206_3216Metric_Pad1.33x1.80mm_HandSolder, F.Cu at (74.9, 83.8)
- added C3: C, Capacitor_SMD:C_1206_3216Metric_Pad1.33x1.80mm_HandSolder, F.Cu at (94.0, 76.8)
- added C4: 100n, Capacitor_SMD:C_1206_3216Metric_Pad1.33x1.80mm_HandSolder, F.Cu at (87.3, 94.8)
- added D5: ACSC02-41SURKWA-F01, fram-prototype:ACSC02-41SURKWA-F01, F.Cu at (127.3, 69.8)
- added J2: AVR-ISP-6, Connector_PinHeader_2.54mm:PinHeader_2x03_P2.54mm_Vertical, F.Cu at (139.7, 83.8)
- added PS1: VXO7805-500-M, fram-prototype:CONV_VXO7805-500-M, F.Cu at (65.4, 79.4)
- added R1: 470, Resistor_SMD:R_1206_3216Metric_Pad1.30x1.75mm_HandSolder, F.Cu at (69.2, 90.8)
- added R2: R_US, Resistor_SMD:R_1206_3216Metric_Pad1.30x1.75mm_HandSolder, F.Cu at (83.2, 72.4)
- added U1: ATmega328-PU, Package_DIP:DIP-28_W7.62mm, F.Cu at (132.1, 82.5)
- added U3: MAX6951, Package_SO:QSOP-16_3.9x4.9mm_P0.635mm, F.Cu at (91.4, 70.8)
- D1: value ACSC02-41SURKWA-F01 -> LED; footprint fram-prototype:ACSC02-41SURKWA-F01 -> LED_SMD:LED_1206_3216Metric_Pad1.42x1.75mm_HandSolder
- U2: value MAX6951 -> MB85RS256B; footprint Package_SO:QSOP-16_3.9x4.9mm_P0.635mm -> Package_SO:SOP-8_5.28x5.23mm_P1.27mm
- moved D1 44.0 mm to (62.9, 90.8)
- moved U2 34.2 mm to (85.1, 102.9)
- moved G*** 30.5 mm to (73.7, 114.3)
- moved D3 4.74 mm to (112.1, 69.8)
- moved D2 4.74 mm to (104.5, 69.8)
- moved D4 4.74 mm to (119.7, 69.8)
Connections:
- D1 pad 1: (no net) -> GND
- D1 pad 2: (no net) -> Net-(D1-Pad2)
- D2 pad 1: (no net) -> /7seg/SEG4
- D2 pad 10: (no net) -> /7seg/SEG2
- D2 pad 2: (no net) -> /7seg/SEG5
- D2 pad 3: (no net) -> /7seg/SEG0
- D2 pad 4: (no net) -> /7seg/SEG6
- D2 pad 5: (no net) -> /7seg/SEG1
- D2 pad 6: (no net) -> /7seg/SEG7
- D2 pad 7: (no net) -> /7seg/SEG8
- D2 pad 8: (no net) -> /7seg/SEG0
- D2 pad 9: (no net) -> /7seg/SEG3
- D3 pad 1: (no net) -> /7seg/SEG4
- D3 pad 10: (no net) -> /7seg/SEG2
- D3 pad 2: (no net) -> /7seg/SEG5
- D3 pad 3: (no net) -> /7seg/SEG1
- D3 pad 4: (no net) -> /7seg/SEG6
- D3 pad 5: (no net) -> /7seg/SEG0
- D3 pad 6: (no net) -> /7seg/SEG7
- D3 pad 7: (no net) -> /7seg/SEG8
- D3 pad 8: (no net) -> /7seg/SEG1
- D3 pad 9: (no net) -> /7seg/SEG3
- D4 pad 1: (no net) -> /7seg/SEG4
- D4 pad 10: (no net) -> /7seg/SEG1
- D4 pad 2: (no net) -> /7seg/SEG5
- D4 pad 3: (no net) -> /7seg/SEG2
- D4 pad 4: (no net) -> /7seg/SEG6
- D4 pad 5: (no net) -> /7seg/SEG0
- D4 pad 6: (no net) -> /7seg/SEG7
- D4 pad 7: (no net) -> /7seg/SEG8
- D4 pad 8: (no net) -> /7seg/SEG2
- D4 pad 9: (no net) -> /7seg/SEG3
- J1 pad 1: (no net) -> +VDC
- SW1 pad A: (no net) -> Net-(SW1-PadA)
- SW1 pad B: (no net) -> Net-(SW1-PadB)
- SW1 pad C: (no net) -> GND
- SW1 pad S1: (no net) -> Net-(SW1-PadS1)
- SW1 pad S2: (no net) -> Net-(SW1-PadS2)
- U2 pad 1: (no net) -> Net-(U2-Pad1)
- U2 pad 2: (no net) -> Net-(U2-Pad2)
- U2 pad 3: (no net) -> Net-(U2-Pad3)
- U2 pad 4: (no net) -> Net-(U2-Pad4)
- U2 pad 5: (no net) -> Net-(U2-Pad5)
- U2 pad 6: (no net) -> Net-(U2-Pad6)
- U2 pad 7: (no net) -> Net-(U2-Pad7)
- U2 pad 8: (no net) -> Net-(U2-Pad8)
Routing:
- net +5V: track 0.00 -> 76.3 mm
- net /7seg/SEG1: track 0.00 -> 72.6 mm, vias 0 -> 5
- net /7seg/SEG8: track 0.00 -> 65.8 mm, vias 0 -> 5
- net /7seg/SEG0: track 0.00 -> 64.5 mm, vias 0 -> 5
- net /7seg/SEG3: track 0.00 -> 61.9 mm, vias 0 -> 5
- net /7seg/SEG4: track 0.00 -> 61.8 mm, vias 0 -> 5
- net /7seg/SEG6: track 0.00 -> 59.8 mm, vias 0 -> 6
- net /7seg/SEG2: track 0.00 -> 58.6 mm, vias 0 -> 5
- net /7seg/SEG7: track 0.00 -> 56.9 mm, vias 0 -> 6
- net /7seg/SEG5: track 0.00 -> 49.6 mm, vias 0 -> 5
- net +VDC: track 0.00 -> 19.9 mm
- net /7seg/DIN: track 0.00 -> 7.66 mm, vias 0 -> 1
- net /7seg/CLK: track 0.00 -> 5.52 mm, vias 0 -> 1
- net Net-(R2-Pad1): track 0.00 -> 4.05 mm
- net Net-(D1-Pad2): track 0.00 -> 3.31 mm
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Other:
- net class 7seg added: clearance 0.0762, trace_width 0.381, via_dia 0.635, via_drill 0.4
- net class Default: clearance 0.2 -> 0.381; trace_width 0.25 -> 0.889
- rule trace_clearance: 0.2 -> 0.381
- board text added: "FRAM PROTOTYPE"
- board text added: "POWER"
