File: fram-prototype.sch (KiCad schematic (older format))
At the start: 8 parts, among them J1 Barrel_Jack, SW1 Rotary_Encoder_Switch, U1 MB85RS256B, U2 MAX6951

Commit message: first basic prototype
Parts:
- removed D1, D2, D3, D4: ACSC02-41SURKWA-F01, fram-prototype:ACSC02-41SURKWA-F01, symbol ACSC02-41SURKWA-F01:ACSC02-41SURKWA-F01
- removed U2: MAX6951, Package_SO:QSOP-16_3.9x4.9mm_P0.635mm, symbol MAX6951:MAX6951
- added C1: 10u, Capacitor_SMD:C_1206_3216Metric_Pad1.33x1.80mm_HandSolder, symbol Device:C
- added C2: 22u, Capacitor_SMD:C_1206_3216Metric_Pad1.33x1.80mm_HandSolder, symbol Device:C
- added C5, C6, C?: C, symbol Device:C
- added D1: LED, LED_SMD:LED_1206_3216Metric_Pad1.42x1.75mm_HandSolder, symbol Device:LED
- added J2: AVR-ISP-6, Connector_PinHeader_2.54mm:PinHeader_2x03_P2.54mm_Vertical, symbol Connector:AVR-ISP-6
- added PS1: VXO7805-500-M, CONV_VXO7805-500-M, symbol VXO7805-500-M:VXO7805-500-M
- added R1: 470, Resistor_SMD:R_1206_3216Metric_Pad1.30x1.75mm_HandSolder, symbol Device:R_US
- added R3, R4: R_US, symbol Device:R_US
- added U1: ATmega328-PU, Package_DIP:DIP-28_W7.62mm, symbol MCU_Microchip_ATmega:ATmega328-PU
- added Y1: Crystal, symbol Device:Crystal
- U2: renamed from U1; footprint (none) -> Package_SO:SOP-8_5.28x5.23mm_P1.27mm
Connections:
- net GND: now also SW1.C, C1.2, C2.2, C5.1, C6.1, C?.1, D1.1 (K), J2.6 (GND), PS1.2 (GND), U1.22 (GND), U1.8 (GND)
- net +VDC: now reaches J1.1
- net +VDC: now also C1.1, PS1.1 (+VIN)
- net at SW1.A: now also U1.2 (PD0)
- net at SW1.B: now also U1.3 (PD1)
- new net: D1.2 (A), R1.2
- new net: J2.5 (~RST), R4.2, U1.1 (~RESET~/PC6)
- new net: C6.2, R3.2, U1.10 (XTAL2/PB7), Y1.2
- new net: C5.2, R3.1, U1.9 (XTAL1/PB6), Y1.1
- new net +5V: C2.1, C?.2, J2.2 (VCC), PS1.3 (+VO), R1.1, R4.1, U1.7 (VCC)
- new net MISO: J2.1 (MISO)
- new net MOSI: J2.4 (MOSI)
- new net SCK: J2.3 (SCK)
- no-connect marks 0 -> 8
Other:
- note added: "POWER"
- note added: "POWER INDICATOR"
- note added: "TODO:\nCHECK SERIAL PIN ASSIGNMENTS"
- moved on the sheet: J1, SW1, U2
