File: kicad/7seg.sch (KiCad schematic (older format))
At the start: 8 parts, among them U3 MAX6951

Commit message: 3v3
Connections:
- net +5V: no longer U3.16 (V+)
- new net +3V3: U3.16 (V+)
Changed lines of the file:
@@
-$EndComp
-$Comp
-L power:+5V #PWR0112
-U 1 1 6010D4FB
-P 3750 1250
-F 0 "#PWR0112" H 3750 1100 50  0001 C CNN
-F 1 "+5V" H 3765 1423 50  0000 C CNN
-F 2 "" H 3750 1250 50  0001 C CNN
-F 3 "" H 3750 1250 50  0001 C CNN
-	1    3750 1250
-	1    0    0    -1
 $EndComp
 $Comp
@@
 	1    0    0    -1
 $EndComp
+$Comp
+L power:+3.3V #PWR0124
+U 1 1 608D6F5A
+P 3750 1250
+F 0 "#PWR0124" H 3750 1100 50  0001 C CNN
+F 1 "+3.3V" H 3765 1423 50  0000 C CNN
+F 2 "" H 3750 1250 50  0001 C CNN
+F 3 "" H 3750 1250 50  0001 C CNN
+	1    3750 1250
+	1    0    0    -1
+$EndComp

Commit message: revA
Connections:
- net +5V is gone; now on net +3V3: C4.1
Changed lines of the file:
@@
 Sheet 2 2
 Title "FRAM Prototype"
-Date "2021-01-26"
-Rev "1.0.0"
+Date "2021-05-03"
+Rev "A"
 Comp "University of Wisconsin-Madison"
 Comment1 "Department of Chemistry"
@@
 $EndComp
 $Comp
-L power:+5V #PWR0116
-U 1 1 60147DC7
-P 4150 2650
-F 0 "#PWR0116" H 4150 2500 50  0001 C CNN
-F 1 "+5V" H 4165 2823 50  0000 C CNN
-F 2 "" H 4150 2650 50  0001 C CNN
-F 3 "" H 4150 2650 50  0001 C CNN
-	1    4150 2650
-	1    0    0    -1
-$EndComp
-$Comp
 L power:+3.3V #PWR0124
 U 1 1 608D6F5A
@@
 	1    0    0    -1
 $EndComp
+$Comp
+L power:+3.3V #PWR0116
+U 1 1 60910A93
+P 4150 2650
+F 0 "#PWR0116" H 4150 2500 50  0001 C CNN
+F 1 "+3.3V" H 4165 2823 50  0000 C CNN
+F 2 "" H 4150 2650 50  0001 C CNN
+F 3 "" H 4150 2650 50  0001 C CNN
+	1    4150 2650
+	1    0    0    -1
+$EndComp
