File: kicad/fram-prototype.kicad_pcb (KiCad board)
At the start: 2 copper layers, 91.4 x 66 mm, 23 parts, among them J1 Barrel_Jack, J2 AVR-ISP-6, SW1 Rotary_Encoder_Switch, U1 ATmega328-PU, U2 MB85RS256B, U3 MAX6951

Commit message: 3v3
Parts:
- added C5: 20p, Capacitor_SMD:C_1206_3216Metric_Pad1.33x1.80mm_HandSolder, F.Cu at (153.7, 72.4)
- added C6: 20p, Capacitor_SMD:C_1206_3216Metric_Pad1.33x1.80mm_HandSolder, F.Cu at (166.6, 65.7)
- added C7: 100n, Capacitor_SMD:C_1206_3216Metric_Pad1.33x1.80mm_HandSolder, F.Cu at (159.7, 72.4)
- added D6: CDBHM260L-HF, footprints:SOP10P27X11-4N, F.Cu at (25.4, 102.9)
- added R3: 1M, Resistor_SMD:R_1206_3216Metric_Pad1.30x1.75mm_HandSolder, F.Cu at (166.6, 69.1)
- added R4: 4.7k, Resistor_SMD:R_1206_3216Metric_Pad1.30x1.75mm_HandSolder, F.Cu at (165.7, 72.4)
- added Y1: 8MHz, Crystal:Crystal_HC49-U_Vertical, F.Cu at (154.7, 67.4)
- PS1: value VXO7805-500-M -> VXO7803-500-M; footprint fram-prototype:CONV_VXO7805-500-M -> footprints:CONV_VXO7805-500-M
- R1: value 470 -> 100
Connections:
- C2 pad 1: +5V -> +3V3
- C4 pad 1: +5V -> (no net)
- J1 pad 1: +VDC -> Net-(D6-Pad3)
- J1 pad 2: GND -> Net-(D6-Pad4)
- J2 pad 2: +5V -> +3V3
- PS1 pad 3: +5V -> +3V3
- PS1 pad 4: Net-(PS1-Pad4) -> (no net)
- R1 pad 1: +5V -> +3V3
- SW1 pad S1: Net-(SW1-PadS1) -> (no net)
- SW1 pad S2: Net-(SW1-PadS2) -> (no net)
- U1 pad 11: Net-(U1-Pad11) -> (no net)
- U1 pad 12: Net-(U1-Pad12) -> (no net)
- U1 pad 13: Net-(U1-Pad13) -> (no net)
- U1 pad 14: Net-(U1-Pad14) -> (no net)
- U1 pad 16: Net-(U1-Pad16) -> /7seg/~CS~
- U1 pad 17: Net-(U1-Pad17) -> SCK
- U1 pad 18: Net-(U1-Pad18) -> MISO
- U1 pad 19: Net-(U1-Pad19) -> MOSI
- U1 pad 20: Net-(U1-Pad20) -> (no net)
- U1 pad 21: Net-(U1-Pad21) -> (no net)
- U1 pad 23: Net-(U1-Pad23) -> (no net)
- U1 pad 24: Net-(U1-Pad24) -> (no net)
- U1 pad 25: Net-(U1-Pad25) -> (no net)
- U1 pad 26: Net-(U1-Pad26) -> (no net)
- U1 pad 27: Net-(U1-Pad27) -> (no net)
- U1 pad 28: Net-(U1-Pad28) -> (no net)
- U1 pad 4: Net-(U1-Pad4) -> (no net)
- U1 pad 5: Net-(U1-Pad5) -> (no net)
- U1 pad 6: Net-(U1-Pad6) -> (no net)
- U1 pad 7: +5V -> +3V3
- U2 pad 1: Net-(U2-Pad1) -> Net-(U1-Pad15)
- U2 pad 2: Net-(U2-Pad2) -> MISO
- U2 pad 3: Net-(U2-Pad3) -> (no net)
- U2 pad 4: Net-(U2-Pad4) -> GND
- U2 pad 5: Net-(U2-Pad5) -> MOSI
- U2 pad 6: Net-(U2-Pad6) -> SCK
- U2 pad 7: Net-(U2-Pad7) -> +3V3
- U2 pad 8: Net-(U2-Pad8) -> +3V3
- U3 pad 1: /7seg/DIN -> MOSI
- U3 pad 16: +5V -> +3V3
- U3 pad 2: /7seg/CLK -> SCK
Routing:
- net +5V: track 76.3 -> 0.00 mm
- net +3V3: track 0.00 -> 76.3 mm
- net MOSI: track 0.00 -> 7.66 mm, vias 0 -> 1
- net /7seg/DIN: track 7.66 -> 0.00 mm, vias 1 -> 0
- net SCK: track 0.00 -> 5.52 mm, vias 0 -> 1
- net /7seg/CLK: track 5.52 -> 0.00 mm, vias 1 -> 0
Other:
- board text added: "RECHECK FOOTPRINT"

Commit message: revA
Parts:
- D6: footprint footprints:SOP10P27X11-4N -> footprints:SOIC245P670X290-4N
- moved C7 69.3 mm to (90.8, 80.0), turned to 270 degrees
- moved R3 66.1 mm to (101.6, 81.3), turned to 90 degrees
- moved D6 50.7 mm to (65.4, 71.8)
- moved C6 46.6 mm to (121.9, 78.7), turned to 180 degrees
- moved Y1 44.3 mm to (112.4, 80.6), turned to 180 degrees
- moved R4 39.2 mm to (128.9, 86.0), turned to 90 degrees
- moved C5 33.3 mm to (121.9, 82.5), turned to 180 degrees
- moved C4 32.8 mm to (97.2, 63.5), turned to 90 degrees
- moved U1 15.7 mm to (116.8, 86.4)
- moved D1 10.8 mm to (63.5, 101.6)
- moved R1 10.8 mm to (69.8, 101.6)
- moved C1 10.6 mm to (61.6, 78.7)
- moved C2 9.53 mm to (74.9, 93.3)
- moved PS1 9.53 mm to (65.4, 88.9)
- moved J2 7.41 mm to (133.3, 87.6)
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Connections:
- C4 pad 1: (no net) -> +3V3
- R4 pad 1: +3V3 -> Net-(J2-Pad5)
- R4 pad 2: Net-(J2-Pad5) -> +3V3
Routing:
- net SCK: track 5.52 -> 106.3 mm, vias 1 -> 2
- net MOSI: track 7.66 -> 100.7 mm
- net +3V3: track 76.3 -> 139.9 mm, vias 0 -> 1
- net MISO: track 0.00 -> 60.6 mm, vias 0 -> 2
- net /7seg/~CS~: track 0.00 -> 46.4 mm, vias 0 -> 1
- net Net-(C6-Pad2): track 0.00 -> 30.3 mm
- net Net-(C5-Pad2): track 0.00 -> 27.0 mm
- net Net-(SW1-PadA): track 0.00 -> 21.4 mm
- net Net-(SW1-PadB): track 0.00 -> 20.2 mm
- net Net-(J2-Pad5): track 0.00 -> 19.6 mm
- net Net-(D6-Pad4): track 0.00 -> 17.7 mm
- net Net-(D6-Pad3): track 0.00 -> 13.0 mm
- net Net-(U1-Pad15): track 0.00 -> 8.87 mm
- net /7seg/SEG5: track 49.6 -> 55.2 mm
- net +VDC: track 19.9 -> 14.4 mm
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Other:
- net class 7seg removed
- net class data added: clearance 0.0762, trace_width 0.381, via_dia 0.635, via_drill 0.4
- board text added: "3.3V ONLY"
- board text added: "9 to 30V"
- board text added: "BLAISE THOMPSON UW MADISON INSTRUMENT SHOP"
- board text added: "REVISION A MAY 2021"
- board text removed: "9 to 30V DC CENTER POSITIVE"
- board text removed: "RECHECK FOOTPRINT"
