File: kicad/fram-prototype.sch (KiCad schematic (older format))
At the start: 16 parts, among them J1 Barrel_Jack, J2 AVR-ISP-6, SW1 Rotary_Encoder_Switch, U1 ATmega328-PU, U2 MB85RS256B, Y1 Crystal

Commit message: 3v3
Parts:
- added D6: CDBHM260L-HF, footprints:SOP10P27X11-4N, symbol Device:D_Bridge_+-AA
- C5, C6: value C -> 20p; footprint (none) -> Capacitor_SMD:C_1206_3216Metric_Pad1.33x1.80mm_HandSolder
- C7: renamed from C?; value C -> 100n; footprint (none) -> Capacitor_SMD:C_1206_3216Metric_Pad1.33x1.80mm_HandSolder
- PS1: value VXO7805-500-M -> VXO7803-500-M
- R1: value 470 -> 100
- R3: value R_US -> 1M; footprint (none) -> Resistor_SMD:R_1206_3216Metric_Pad1.30x1.75mm_HandSolder
- R4: value R_US -> 4.7k; footprint (none) -> Resistor_SMD:R_1206_3216Metric_Pad1.30x1.75mm_HandSolder
- Y1: value Crystal -> 8MHz; footprint (none) -> Crystal:Crystal_HC49-U_Vertical
Connections:
- net +5V is gone; now on net +3V3: C2.1, C7.2, J2.2 (VCC), PS1.3 (+VO), R1.1, R4.1, U1.7 (VCC)
- net +VDC: now also D6.1 (+); no longer J1.1
- net 7seg/~CS~: now also U1.16 (PB2)
- net GND: now also U2.4 (GND), D6.2 (-); no longer J1.2
- net MISO: now also U1.18 (PB4), U2.2 (SO)
- net MOSI: now also U1.19 (PB5), U2.5 (SI)
- net SCK: now also U1.17 (PB3), U2.6 (SCK)
- net at U2.1 (~CS): now also U1.15 (PB1)
- net +3V3: now reaches U2.7 (~HOLD)
- net +3V3: now also U2.8 (VDD)
- new net: D6.3 (~~), J1.1
- new net: D6.4 (~~), J1.2
- no-connect marks 8 -> 19
Other:
- note added: "5 to 35 V\nAC or DC\n"
- note added: "POWER INDICATOR (RED)"
- note removed: "POWER INDICATOR"
- note removed: "TODO:\nCHECK SERIAL PIN ASSIGNMENTS"
- moved on the sheet: C1, C2, D1, PS1, R1

Commit message: revA
Parts:
- D6: footprint footprints:SOP10P27X11-4N -> footprints:SOIC245P670X290-4N
Connections:
- net +3V3: now also R4.2; no longer R4.1
- net at J2.5 (~RST), U1.1 (~RESET~/PC6): now also R4.1; no longer R4.2
Changed lines of the file:
@@
 F 3 "~" H 5900 3050 50  0001 C CNN
 	1    5900 3050
-	1    0    0    -1
+	-1   0    0    1
 $EndComp
 NoConn ~ 2600 1700
@@
 Text GLabel 2600 2200 2    50   Output ~ 0
 MOSI
-Connection ~ 5900 3200
-Wire Wire Line
-	5900 3200 6500 3200
-Wire Wire Line
-	2600 3200 5900 3200
 Wire Wire Line
 	2600 3500 6000 3500
@@
 F 0 "D6" H 2250 6850 50  0000 L CNN
 F 1 "CDBHM260L-HF" H 2000 7200 50  0000 L CNN
-F 2 "footprints:SOP10P27X11-4N" H 2300 6850 50  0001 C CNN
+F 2 "footprints:SOIC245P670X290-4N" H 2300 6850 50  0001 C CNN
 F 3 "~" H 2300 6850 50  0001 C CNN
 	1    2300 6850
@@
 	1    0    0    1
 $EndComp
+Wire Wire Line
+	2600 3200 5900 3200
+Connection ~ 5900 3200
+Wire Wire Line
+	5900 3200 6500 3200
 $EndSCHEMATC
